File: Hardware/KiCAD/JunketOnSteroidsTTGO.kicad_pcb (KiCad board)
At the start: 2 copper layers, 52.1 x 26.7 mm, 29 parts, among them J1 To PSU host board, J2 To PSU host board, J3 Serial, J4 ESP32-TFT, J5 ESP32-TFT, J6 NRST/SWIM

Commit message: Swap GPIO12 & 15, Add !ON with solder-option, Replace SWIM with I2C
Parts:
- added JP2: ON/SW, Jumper:SolderJumper-3_P1.3mm_Open_RoundedPad1.0x1.5mm, B.Cu at (112.4, 80.6)
- added R4: 2k2, Resistor_THT:R_Axial_DIN0204_L3.6mm_D1.6mm_P7.62mm_Horizontal, F.Cu at (118.7, 82.5)
- J6: value NRST/SWIM -> I2C
- JP1: moved to B.Cu
- moved C2 20.7 mm to (146.1, 81.3)
- moved JP1 20.7 mm to (148.0, 75.6)
- moved C11 20.7 mm to (120.0, 70.5)
- moved C31 20.7 mm to (120.0, 79.4)
- moved J4 20.7 mm to (136.5, 65.4)
- moved J5 20.7 mm to (136.5, 88.3)
- moved R11 20.7 mm to (116.2, 68.6)
- moved R12 20.7 mm to (116.2, 70.5)
- moved R2 20.7 mm to (106.0, 65.4)
- moved R31 20.7 mm to (116.2, 77.5)
- moved R32 20.7 mm to (116.2, 79.4)
- moved C1 20.7 mm to (147.3, 68.6)
- moved C21 20.7 mm to (120.0, 74.9)
- moved C3 20.7 mm to (135.3, 68.6)
- moved FID1 20.7 mm to (103.5, 88.3)
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Connections:
- J1 pad 6: Net-(J1-Pad6) -> /!ON
- J1 pad 7: Net-(J1-Pad7) -> /FAN
- J4 pad 3: Net-(J4-Pad3) -> /GPIO27
- J5 pad 10: Net-(J5-Pad10) -> /SDA
- J5 pad 4: Net-(J5-Pad4) -> /FAN
- J5 pad 5: Net-(J5-Pad5) -> /GPIO13
- J5 pad 6: /GPIO12 -> /GPIO15
- J5 pad 7: /GPIO15 -> /ADC12
- J5 pad 8: /ADC12 -> Net-(J5-Pad8)
- J5 pad 9: Net-(J5-Pad9) -> /SCL
- J6 pad 1: +3V3 -> /GND
- J6 pad 2: /SWIM -> /SDA
- J6 pad 3: /GND -> /SCL
- J6 pad 4: /NRST -> +3V3
- R41 pad 2: /GPIO15 -> /GPIO13
- R51 pad 2: /GPIO12 -> /GPIO15
Routing:
- net /GPIO27: track 0.00 -> 30.8 mm
- net /FAN: track 0.00 -> 27.5 mm
- net /GND: track 164.0 -> 140.4 mm, vias 0 -> 1
- net /GPIO12: track 17.1 -> 0.00 mm
- net +3V3: track 63.5 -> 49.8 mm
- net /GPIO13: track 0.00 -> 12.5 mm
- net /!ON: track 0.00 -> 8.89 mm
- net Net-(JP2-Pad3): track 0.00 -> 8.18 mm
- net /ADC12: track 18.8 -> 21.3 mm
- net GNDD: track 7.82 -> 6.89 mm
Other:
- board text added: "+5V TX GND RX"
- board text added: "12 34"
- board text added: "GND SDA SLC +3V3"
- board text added: "Rev 0.2"
- board text added: "SW ON"
- board text removed: "Rev 0.1"

Commit message: Rev 0.3
Parts:
- added JP3: Vin_sense, Jumper:SolderJumper-3_P1.3mm_Open_RoundedPad1.0x1.5mm, B.Cu at (112.4, 71.8)
- added TP1: Vin_sense, Connector_Wire:SolderWire-0.1sqmm_1x01_D0.4mm_OD1mm, F.Cu at (105.4, 65.4)
- J3, J6: footprint Connector_PinHeader_2.54mm:PinHeader_1x04_P2.54mm_Vertical -> Connector_PinHeader_2.54mm:PinHeader_1x04_P2.54mm_Horizontal
- moved J3 7.62 mm to (141.6, 65.4), turned to 90 degrees
- moved R34 3.17 mm to (106.0, 68.6)
- renumbered R2 to R34, R4 to R6
Connections:
- J6 pad 1: /GND -> +3V3
- J6 pad 2: /SDA -> /GND
- J6 pad 4: +3V3 -> /SDA
- R31 pad 2: /Vin_sense -> Net-(JP3-Pad2)
- R34 pad 2: /Vin_sense -> Net-(JP3-Pad3)
Routing:
- net /SCL: track 0.00 -> 29.9 mm
- net /SDA: track 0.00 -> 29.3 mm
- net +3V3: track 49.8 -> 63.5 mm
- net Net-(JP3-Pad2): track 0.00 -> 13.3 mm
- net /GND: track 140.4 -> 153.0 mm
- net Net-(JP3-Pad3): track 0.00 -> 9.12 mm
- net /Vin: track 0.00 -> 3.44 mm
- net /FAN: track 27.5 -> 29.5 mm
- net /Iout_sense: track 5.34 -> 7.09 mm
- net /GPIO27: track 30.8 -> 29.8 mm
- net /Vin_sense: track 9.46 -> 10.2 mm
Other:
- board text added: "3V3 GND SCL SDA"
- board text added: "Rev 0.3"
- board text removed: "GND SDA SLC +3V3"
- board text removed: "Rev 0.2"
