File: Hardware/KiCAD/JuntekOnSteroidsTTGO.kicad_pcb (KiCad board)
At the start: 2 copper layers, 52.1 x 26.7 mm, 33 parts, among them J1 To PSU host board, J2 To PSU host board, J3 Serial, J4 ESP32-TFT, J5 ESP32-TFT, J6 I2C

Commit message: Tidy I2C bits
Parts:
- J6: moved to B.Cu
- moved J6 7.62 mm to (141.6, 88.3)
Connections:
- J6 pad 1: +3V3 -> /SDA
- J6 pad 2: /GND -> /SCL
- J6 pad 3: /SCL -> /GND
- J6 pad 4: /SDA -> +3V3
Routing:
- net /SDA: track 29.3 -> 41.3 mm
- net /SCL: track 29.9 -> 39.3 mm
- net /GND: track 153.0 -> 158.7 mm
- net +3V3: track 63.5 -> 68.8 mm
Other:
- board text added: "All 4 traces to all 4 pins to enable choice of I2C pinout standard. E.g. DFRobot vs [Grove, Crowtail, QWIIC, nodeLynk, STEMMA(QT)] Not inc. Quick2Wire & BreakoutGarden"
- board text added: "I2C"
- board text added: "Rev 0.5"
- board text removed: "3V3 GND SCL SDA"
- board text removed: "Rev 0.4"
