File: Hardware/KiCAD/JuntekOnSteroidsTTGO.sch (KiCad schematic (older format))
At the start: 33 parts, among them J1 To PSU host board, J2 To PSU host board, J3 Serial, J4 ESP32-TFT, J5 ESP32-TFT, J6 I2C

Commit message: Tidy I2C bits
Connections:
- net +3V3: now also J6.4 (Pin_4); no longer J6.1 (Pin_1)
- net GND: now also J6.3 (Pin_3); no longer J6.2 (Pin_2)
- net SCL: now also J6.2 (Pin_2); no longer J6.3 (Pin_3)
- net SDA: now also J6.1 (Pin_1); no longer J6.4 (Pin_4)
Changed lines of the file:
@@
 Sheet 1 1
 Title "Drok/Juntek-on-steroids"
-Date "2021-03-21"
-Rev "0.4"
+Date "2021-05-03"
+Rev "0.5"
 Comp ""
 Comment1 ""
@@
 L Connector_Generic:Conn_01x04 J6
 U 1 1 60548EC3
-P 4100 3950
-F 0 "J6" V 4100 4100 50  0000 L CNN
-F 1 "I2C" V 4200 3700 50  0000 L CNN
-F 2 "Connector_PinHeader_2.54mm:PinHeader_1x04_P2.54mm_Horizontal" H 4100 3950 50  0001 C CNN
-F 3 "~" H 4100 3950 50  0001 C CNN
-	1    4100 3950
-	0    1    1    0
+P 4000 3950
+F 0 "J6" V 4000 4100 50  0000 L CNN
+F 1 "I2C" V 4100 3700 50  0000 L CNN
+F 2 "Connector_PinHeader_2.54mm:PinHeader_1x04_P2.54mm_Horizontal" H 4000 3950 50  0001 C CNN
+F 3 "~" H 4000 3950 50  0001 C CNN
+	1    4000 3950
+	0    -1   1    0
 $EndComp
 Text Label 4050 2950 0    50   ~ 0
