File: Hardware/KiCAD/JuntekOnSteroidsTTGO.sch (KiCad schematic (older format))
At the start: 29 parts, among them J1 To PSU host board, J2 To PSU host board, J3 Serial, J4 ESP32-TFT, J5 ESP32-TFT, J6 I2C, J7 PWR, J8 Conn_02x12_Odd_Even

Commit message: Change exp. connector, add ADC caps
Parts:
- added C1, C2, C3, C4: 0.1µ, Capacitor_THT:C_Disc_D3.0mm_W1.6mm_P2.50mm, symbol Device:C
- added TP3: ADC2, Connector_Wire:SolderWire-0.1sqmm_1x01_D0.4mm_OD1mm, symbol Connector:TestPoint
- C8: footprint Capacitor_THT:C_Disc_D4.7mm_W2.5mm_P5.00mm -> Capacitor_THT:C_Disc_D3.0mm_W1.6mm_P2.50mm
- J8: footprint Connector_IDC:IDC-Header_2x12_P2.54mm_Vertical -> Connector_PinHeader_2.54mm:PinHeader_2x12_P2.54mm_Horizontal
Connections:
- net ADC1: now also TP3.1
Other:
- moved on the sheet: TP1
Changed lines of the file:
@@
 	1    0    0    -1
 $EndComp
-Text Label 4250 1700 0    50   ~ 0
+Text Label 4250 1600 0    50   ~ 0
 ADC0
 $Comp
@@
 L Connector:TestPoint TP1
 U 1 1 60589602
-P 4250 1700
-F 0 "TP1" V 4250 1950 50  0000 C CNN
-F 1 "ADC0" V 4350 1950 50  0000 C CNN
-F 2 "Connector_Wire:SolderWire-0.1sqmm_1x01_D0.4mm_OD1mm" H 4450 1700 50  0001 C CNN
-F 3 "~" H 4450 1700 50  0001 C CNN
-	1    4250 1700
+P 4250 1600
+F 0 "TP1" V 4250 1850 50  0000 C CNN
+F 1 "ADC0" V 4350 1850 50  0000 C CNN
+F 2 "Connector_Wire:SolderWire-0.1sqmm_1x01_D0.4mm_OD1mm" H 4450 1600 50  0001 C CNN
+F 3 "~" H 4450 1600 50  0001 C CNN
+	1    4250 1600
 	0    -1   -1   0
 $EndComp
@@
 F 0 "C8" H 9100 2950 50  0000 L CNN
 F 1 "0.1µ" H 9100 3100 50  0000 L CNN
-F 2 "Capacitor_THT:C_Disc_D4.7mm_W2.5mm_P5.00mm" H 9288 2700 50  0001 C CNN
+F 2 "Capacitor_THT:C_Disc_D3.0mm_W1.6mm_P2.50mm" H 9288 2700 50  0001 C CNN
 F 3 "~" H 9250 2850 50  0001 C CNN
 	1    9250 2850
@@
 F 0 "J8" V 5796 1012 50  0000 R CNN
 F 1 "Conn_02x12_Odd_Even" V 5705 1012 50  0000 R CNN
-F 2 "Connector_IDC:IDC-Header_2x12_P2.54mm_Vertical" H 5700 1700 50  0001 C CNN
+F 2 "Connector_PinHeader_2.54mm:PinHeader_2x12_P2.54mm_Horizontal" H 5700 1700 50  0001 C CNN
 F 3 "~" H 5700 1700 50  0001 C CNN
 	1    5700 1700
@@
 	1    0    0    -1
 $EndComp
+$Comp
+L Device:C C1
+U 1 1 60A8437B
+P 7950 1950
+F 0 "C1" H 7800 2050 50  0000 L CNN
+F 1 "0.1µ" H 7800 2200 50  0000 L CNN
+F 2 "Capacitor_THT:C_Disc_D3.0mm_W1.6mm_P2.50mm" H 7988 1800 50  0001 C CNN
+F 3 "~" H 7950 1950 50  0001 C CNN
+	1    7950 1950
+	1    0    0    -1
+$EndComp
+$Comp
+L Device:C C2
+U 1 1 60A8638B
+P 8250 1950
+F 0 "C2" H 8100 2050 50  0000 L CNN
+F 1 "0.1µ" H 8100 2200 50  0000 L CNN
+F 2 "Capacitor_THT:C_Disc_D3.0mm_W1.6mm_P2.50mm" H 8288 1800 50  0001 C CNN
+F 3 "~" H 8250 1950 50  0001 C CNN
+	1    8250 1950
+	1    0    0    -1
+$EndComp
+$Comp
+L Device:C C3
+U 1 1 60A8822B
+P 7950 2500
+F 0 "C3" H 7800 2600 50  0000 L CNN
+F 1 "0.1µ" H 7800 2750 50  0000 L CNN
+F 2 "Capacitor_THT:C_Disc_D3.0mm_W1.6mm_P2.50mm" H 7988 2350 50  0001 C CNN
+F 3 "~" H 7950 2500 50  0001 C CNN
+	1    7950 2500
+	1    0    0    -1
+$EndComp
+$Comp
+L Device:C C4
+U 1 1 60A8A0CB
+P 8250 2500
+F 0 "C4" H 8100 2600 50  0000 L CNN
+F 1 "0.1µ" H 8100 2750 50  0000 L CNN
+F 2 "Capacitor_THT:C_Disc_D3.0mm_W1.6mm_P2.50mm" H 8288 2350 50  0001 C CNN
+F 3 "~" H 8250 2500 50  0001 C CNN
+	1    8250 2500
+	1    0    0    -1
+$EndComp
+$Comp
+L Connector:TestPoint TP3
+U 1 1 60A8AD01
+P 4250 1100
+F 0 "TP3" V 4250 1350 50  0000 C CNN
+F 1 "ADC2" V 4350 1350 50  0000 C CNN
+F 2 "Connector_Wire:SolderWire-0.1sqmm_1x01_D0.4mm_OD1mm" H 4450 1100 50  0001 C CNN
+F 3 "~" H 4450 1100 50  0001 C CNN
+	1    4250 1100
+	0    -1   -1   0
+$EndComp
+Text Label 4250 1100 0    50   ~ 0
+ADC1
 $EndSCHEMATC

Commit message: v2.2
Parts:
- removed J3: Serial, Connector_PinHeader_2.54mm:PinHeader_1x04_P2.54mm_Horizontal, symbol Connector_Generic:Conn_01x04
- removed J6: I2C, Connector_PinHeader_2.54mm:PinHeader_1x04_P2.54mm_Horizontal, symbol Connector_Generic:Conn_01x04
- removed J7: PWR, Connector_PinHeader_2.54mm:PinHeader_1x02_P2.54mm_Horizontal, symbol Connector_Generic:Conn_01x02
- removed J8: Conn_02x12_Odd_Even, Connector_PinHeader_2.54mm:PinHeader_2x12_P2.54mm_Horizontal, symbol Connector_Generic:Conn_02x12_Odd_Even
- removed JP2: Vin_sense, Jumper:SolderJumper-3_P1.3mm_Open_RoundedPad1.0x1.5mm, symbol Jumper:SolderJumper_3_Open
- removed R3, R4, R9: 3M8, Resistor_THT:R_Axial_DIN0204_L3.6mm_D1.6mm_P7.62mm_Horizontal, symbol Device:R
- removed TP1: ADC0, Connector_Wire:SolderWire-0.1sqmm_1x01_D0.4mm_OD1mm, symbol Connector:TestPoint
- removed TP2: ADC1, Connector_Wire:SolderWire-0.1sqmm_1x01_D0.4mm_OD1mm, symbol Connector:TestPoint
- removed TP3: ADC2, Connector_Wire:SolderWire-0.1sqmm_1x01_D0.4mm_OD1mm, symbol Connector:TestPoint
- added J11: Expansion1, Connector_PinHeader_2.54mm:PinHeader_1x12_P2.54mm_Horizontal, symbol Connector_Generic:Conn_01x12
- added J12: Expansion2, Connector_PinHeader_2.54mm:PinHeader_1x12_P2.54mm_Horizontal, symbol Connector_Generic:Conn_01x12
- added J6: feedback, Connector_PinHeader_2.54mm:PinHeader_1x03_P2.54mm_Horizontal, symbol Connector_Generic:Conn_01x03
- added J7: I2C, Connector_JST:JST_PH_B4B-PH-K_1x04_P2.00mm_Vertical, symbol Connector_Generic:Conn_01x04
- added JP1001, JP1002: SolderJumper_2_Open, Jumper:SolderJumper-2_P1.3mm_Open_RoundedPad1.0x1.5mm, symbol Jumper:SolderJumper_2_Open
- added R1001: 10k/none, Resistor_THT:R_Axial_DIN0204_L3.6mm_D1.6mm_P7.62mm_Horizontal, symbol Device:R
- added R1002: 2k2/none, Resistor_THT:R_Axial_DIN0204_L3.6mm_D1.6mm_P7.62mm_Horizontal, symbol Device:R
- added R1003: 1k/zero, Resistor_THT:R_Axial_DIN0204_L3.6mm_D1.6mm_P7.62mm_Horizontal, symbol Device:R
- JP3: value Vin_sense -> VinSense
- JP4: value Vin_sense -> Iout_sense
- JP5: value Vin_sense -> VoutSense
- JP6: value Vin_sense -> FanPWM
- R11: renamed from R2; value 3M8 -> 68k/zero
- R12: renamed from R7; value 3M8 -> 68k/zero
- R14: renamed from R5; value 3M8 -> 1k/zero
- R15: renamed from R6; value 3M8 -> 100k/none
- R17: renamed from R1; value 3M8 -> 1k
Connections:
- net +3V3: now also J11.2 (Pin_2), J7.3 (Pin_3)
- net A0: now also JP4.1 (A)
- net A1: now also JP5.1 (A)
- net A2: now also JP3.1 (A)
- net A3: now also R17.1, J6.2 (Pin_2)
- net ADC0: now also JP5.3 (B)
- net ADC1: now also JP3.3 (B)
- net ADC2: now also J1.7 (Pin_7), JP6.3 (B), J6.1 (Pin_1)
- net ADC3: now also JP4.3 (B)
- net GND: now also C1.2, C2.2, C3.2, C4.2, R15.2, J11.1 (Pin_1), J11.11 (Pin_11), J7.4 (Pin_4), R1001.2, R1002.2
- net GPIO12: now also J11.7 (Pin_7), J6.3 (Pin_3), R1001.1
- net GPIO13: now also J11.6 (Pin_6), JP1002.1 (A)
- net GPIO15: now also R1003.2
- net GPIO17: now also J11.5 (Pin_5), JP1001.1 (A)
- net GPIO2: now also R14.2
- net GPIO25: now also J11.8 (Pin_8)
- net GPIO26: now also J11.9 (Pin_9)
- net GPIO27: now also J11.10 (Pin_10)
- net GPIO32: now also R11.2
- net GPIO33: now also R12.2
- net RX: now also JP1002.2 (B)
- net SCL: now also J11.4 (Pin_4), J7.1 (Pin_1)
- net SDA: now also J11.3 (Pin_3), J7.2 (Pin_2)
- net TX: now also JP1001.2 (B)
- net VCC: now also J11.12 (Pin_12)
- net J1.1: now reaches J1.1 (Pin_1)
- net J1.1: now also C1.1, JP4.2 (C)
- net J1.2: now reaches J1.2 (Pin_2)
- net J1.2: now also C2.1, JP5.2 (C)
- net J1.3: now reaches J1.3 (Pin_3)
- net J1.3: now also C3.1, JP3.2 (C), R15.1
- net J1.4: now reaches J1.4 (Pin_4)
- net J1.4: now also R12.1
- net J1.5: now reaches J1.5 (Pin_5)
- net J1.5: now also R11.1
- net J1.6: now reaches J1.6 (Pin_6)
- net J1.6: now also R14.1, R1002.1
- net J1.8: now reaches J1.8 (Pin_8)
- net J1.8: now also JP6.1 (A)
- net at JP6.2 (C): now also R1003.1
- net IloadSense: now reaches C4.1
- net Shunt: now reaches R17.2
- no-connect marks 3 -> 2
Other:
- note added: "VCC = +5Vdc\nSignal lables based on B3603. Other devices need software re-allocation."
- note removed: "VCC = +5Vdc"
- moved on the sheet: C1, C2, C3, C4, C7, C8, FID1, FID2, FID3, J1, J2, J4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

Commit message: v2.2 and a bit
Parts:
- added R1004: 100k/zero, Resistor_THT:R_Axial_DIN0204_L3.6mm_D1.6mm_P7.62mm_Horizontal, symbol Device:R
- added R1005: 1k/none, Resistor_THT:R_Axial_DIN0204_L3.6mm_D1.6mm_P7.62mm_Horizontal, symbol Device:R
- R17: value 1k -> 1k/zero
Connections:
- net A3: no longer J6.2 (Pin_2)
- net ADC2: now also R1004.2, R1005.1; no longer J6.1 (Pin_1)
- net GND: now also R1005.2
- net Shunt renamed J6.2
- net J6.2: now also J6.2 (Pin_2)
- new net J6.1: J6.1 (Pin_1), R1004.1
Other:
- moved on the sheet: R17
Changed lines of the file:
@@
 L Device:R R17
 U 1 1 60BC63B7
-P 4150 4650
-F 0 "R17" V 4150 4650 50  0000 C CNN
-F 1 "1k" V 4250 4650 50  0000 C CNN
-F 2 "Resistor_THT:R_Axial_DIN0204_L3.6mm_D1.6mm_P7.62mm_Horizontal" V 4080 4650 50  0001 C CNN
-F 3 "~" H 4150 4650 50  0001 C CNN
-	1    4150 4650
+P 3950 4650
+F 0 "R17" V 3950 4650 50  0000 C CNN
+F 1 "1k/zero" V 4050 4650 50  0000 C CNN
+F 2 "Resistor_THT:R_Axial_DIN0204_L3.6mm_D1.6mm_P7.62mm_Horizontal" V 3880 4650 50  0001 C CNN
+F 3 "~" H 3950 4650 50  0001 C CNN
+	1    3950 4650
 	1    0    0    -1
 $EndComp
@@
 Text Label 8750 5700 3    50   ~ 0
 GPIO17
-Text Label 4150 5900 0    50   ~ 0
+Text Label 3950 5900 0    50   ~ 0
 Shunt
 Text Label 8350 5700 3    50   ~ 0
@@
 $EndComp
 Wire Wire Line
-	4150 4250 4150 4500
-Connection ~ 4150 4250
-Wire Wire Line
-	4150 4250 7100 4250
+	3950 4250 3950 4500
 Wire Wire Line
 	4850 4200 4850 5000
@@
 Wire Wire Line
 	6500 2900 6500 3450
-Connection ~ 4050 4100
-Wire Wire Line
-	4050 4100 6400 4100
-Wire Wire Line
-	3000 4100 4050 4100
+Wire Wire Line
+	3000 4100 3300 4100
 Wire Wire Line
 	4050 2900 4050 2850
@@
 Wire Wire Line
 	4050 3900 4050 3200
-Wire Wire Line
-	4050 4100 4050 5100
-Wire Wire Line
-	2750 5100 4050 5100
-Wire Wire Line
-	3950 5000 3950 4250
-Wire Wire Line
-	3950 4250 4150 4250
 Wire Wire Line
 	2750 5000 3950 5000
@@
 	9450 5650 9450 5700
 Wire Wire Line
-	4150 4800 4150 5900
+	3950 4800 3950 5000
+$Comp
+L Device:R R1004
+U 1 1 611A29B7
+P 3100 5100
+F 0 "R1004" V 3100 5100 50  0000 C CNN
+F 1 "100k/zero" V 3000 5150 50  0000 C CNN
+F 2 "Resistor_THT:R_Axial_DIN0204_L3.6mm_D1.6mm_P7.62mm_Horizontal" V 3030 5100 50  0001 C CNN
+F 3 "~" H 3100 5100 50  0001 C CNN
+	1    3100 5100
+	0    -1   -1   0
+$EndComp
+$Comp
+L Device:R R1005
+U 1 1 611BB67B
+P 3500 5100
+F 0 "R1005" V 3500 5100 50  0000 C CNN
+F 1 "1k/none" V 3400 5100 50  0000 C CNN
+F 2 "Resistor_THT:R_Axial_DIN0204_L3.6mm_D1.6mm_P7.62mm_Horizontal" V 3430 5100 50  0001 C CNN
+F 3 "~" H 3500 5100 50  0001 C CNN
+	1    3500 5100
+	0    -1   -1   0
+$EndComp
+Wire Wire Line
+	2750 5100 2950 5100
+Wire Wire Line
+	3250 5100 3300 5100
+Wire Wire Line
+	3650 5100 3700 5100
+Wire Wire Line
+	3700 5100 3700 5200
+Wire Wire Line
+	3300 5100 3300 4100
+Connection ~ 3300 5100
+Wire Wire Line
+	3300 5100 3350 5100
+Connection ~ 3300 4100
+Wire Wire Line
+	3300 4100 6400 4100
+Text Label 3700 5200 0    50   ~ 0
+GND
+Wire Wire Line
+	3950 4250 7100 4250
+Connection ~ 3950 5000
+Wire Wire Line
+	3950 5000 3950 5900
 $EndSCHEMATC
